Commit message: Make the gripper finger limits symmetric (0.05 m both)
`joint_right` carried `upper="0.0715"` while `joint_left` had `upper="0.05"`,
inherited from the CAD URDF export. The two fingers are driven by a single
RS-00 pinion turning two opposed racks, so their travel is mechanically
identical -- the asymmetry was a CAD artefact, not a property of the machine.

Measured on hardware: driving both fingers out to 40 mm leaves
`|left - right|` at 0.00000 mm across every solver setting swept in
docs/GRIPPER_RESIDUAL_MOTION.md, with backlash of +/-0.37 mm at the jaw. The
coupling is 1:1.

This also makes the asset match its own documentation. The gripper coupling
work described the stroke as symmetric and 1:1 while the shipped USD still
declared 0.0715 on the right finger, so the docs and the data disagreed.

Changed:
  * USD physics layer  -- joint_right upperLimit 0.0715 -> 0.05
  * source URDF        -- joint_right upper 0.0715 -> 0.05
  * VALIDATION.md and its generator -- describe the fingers as mimic-coupled
    with a single stroke, instead of "asymmetric strokes come from CAD"
  * isaacsim_traj_sender.py -- comment referenced the old per-finger limits

The exported MJCF (menagerie PR #300) and the newton-assets package (PR #45)
already used 0.05 on both joints, so this brings the USD in line with them
rather than changing behaviour downstream.

Verified after the change:

  Isaac Sim 6.1  mimic composed True, static 0.00006 mm, slewing 0.00629 mm, PASS
  validate_physics_fidelity.py  failures [], MJCF compiles under mujoco 3.10

File: third_party/reBotArm_control_py/urdf/00-arm-rs_asm-v3/urdf/00-arm-rs_asm-v3.urdf (robot description, URDF)
Before this commit: robot 00-arm-rs_asm-v3, 10 links, 9 joints
Joints:
- joint joint_right: limit lower=0 upper=0.0715 effort=500 velocity=10 -> lower=0 upper=0.05 effort=500 velocity=10
